File: scheme/light-node/light-node.sch (KiCad schematic (older format))
At the start: 18 parts, among them P1 CONN_2, P2 CONN_2, P3 CONN_6, Q1 NPN, SW1 SW_RESET, SW2 SW_PROGRAM, T1 220 VAC 5 VDC, U1 SPX2920M3-3.3, U2 ESP866_ESP-12E

Commit message: light-node: PCB done
Connections:
- net 5Vcc: now also T1.3 (SA); no longer T1.4 (SB)
- net GND: now also T1.4 (SB); no longer T1.3 (SA)
- net AC_L: now reaches RL1.11 (COM)
- net AC_L: now also P1.1 (P1), T1.2 (AB); no longer P2.1 (P1)
- net AC_Lout: now reaches RL1.14 (L2_NO)
- net AC_Lout: now also P2.1 (P1); no longer P2.2 (PM)
- net AC_N: now reaches P1.2 (PM), T1.1 (AA)
- net AC_N: now also P2.2 (PM)
Other:
- moved on the sheet: P2
Changed lines of the file:
@@
 LIBS:relay
 LIBS:esp866_esp-12
-LIBS:transfo
+LIBS:light-node-cache
 EELAYER 27 0
 EELAYER END
@@
 Sheet 1 1
 Title ""
-Date "18 jan 2016"
+Date "19 jan 2016"
 Rev ""
 Comp ""
@@
 Comment4 ""
 $EndDescr
-$Comp
-L RZ03-1C4-D005 RL1
-U 1 1 569CD021
-P 5200 1700
-F 0 "RL1" H 5200 1300 60  0000 C CNN
-F 1 "RZ03-1C4-D005" H 5200 2100 60  0000 C CNN
-F 2 "~" H 5200 2100 60  0000 C CNN
-F 3 "~" H 5200 2100 60  0000 C CNN
-	1    5200 1700
-	1    0    0    -1
-$EndComp
 $Comp
 L ESP866_ESP-12E U2
@@
 L CONN_2 P2
 U 1 1 569CE4CF
-P 6400 1900
-F 0 "P2" V 6350 1900 40  0000 C CNN
-F 1 "CONN_2" V 6450 1900 40  0000 C CNN
-F 2 "" H 6400 1900 60  0000 C CNN
-F 3 "" H 6400 1900 60  0000 C CNN
-	1    6400 1900
+P 5800 2500
+F 0 "P2" V 5750 2500 40  0000 C CNN
+F 1 "CONN_2" V 5850 2500 40  0000 C CNN
+F 2 "" H 5800 2500 60  0000 C CNN
+F 3 "" H 5800 2500 60  0000 C CNN
+	1    5800 2500
 	1    0    0    -1
 $EndComp
@@
 Wire Wire Line
 	1350 1850 1500 1850
+Text Label 2300 1450 0    60   ~ 0
+GND
 Text Label 2300 1850 0    60   ~ 0
-GND
-Text Label 2300 1450 0    60   ~ 0
 5Vcc
-Wire Wire Line
-	2300 1450 2500 1450
-Wire Wire Line
-	2500 1450 2500 1500
-Wire Wire Line
-	2500 1500 2800 1500
-Wire Wire Line
-	2300 1850 2500 1850
-Wire Wire Line
-	2500 1850 2500 1800
-Wire Wire Line
-	2500 1800 3200 1800
 Text Label 3600 1500 0    60   ~ 0
 3.3Vcc
@@
 Text Label 5750 1450 0    60   ~ 0
 5Vcc
-Wire Wire Line
-	4650 1850 4600 1850
-Wire Wire Line
-	4600 1850 4600 2200
-Wire Wire Line
-	4600 2200 5800 2200
-Wire Wire Line
-	5800 2200 5800 1850
 NoConn ~ 4650 1750
 NoConn ~ 5750 1750
@@
 ESP_RX
 Wire Wire Line
-	5750 1850 5950 1850
-Wire Wire Line
-	4650 1950 4650 2150
-Wire Wire Line
-	4650 2150 5750 2150
-Wire Wire Line
-	5750 2150 5750 1950
-Wire Wire Line
-	5950 1850 5950 1800
-Wire Wire Line
-	5950 1800 6050 1800
-Connection ~ 5800 1850
-Wire Wire Line
-	5750 1950 5950 1950
-Wire Wire Line
-	5950 1950 5950 2000
-Wire Wire Line
-	5950 2000 6050 2000
+	2300 1850 2650 1850
+Wire Wire Line
+	2650 1850 2650 1500
+Wire Wire Line
+	2650 1500 2800 1500
+Wire Wire Line
+	2300 1450 2600 1450
+Wire Wire Line
+	2600 1450 2600 1800
+Wire Wire Line
+	2600 1800 3200 1800
+Text Label 1200 1550 0    60   ~ 0
+AC_N
+Text Label 1200 1750 0    60   ~ 0
+AC_L
+Text Label 4650 1850 2    60   ~ 0
+AC_L
+Text Label 5450 2600 2    60   ~ 0
+AC_N
+$Comp
+L RZ03-1C4-D005 RL1
+U 1 1 569CD021
+P 5200 1700
+F 0 "RL1" H 5200 1300 60  0000 C CNN
+F 1 "RZ03-1C4-D005" H 5200 2100 60  0000 C CNN
+F 2 "~" H 5200 2100 60  0000 C CNN
+F 3 "~" H 5200 2100 60  0000 C CNN
+	1    5200 1700
+	1    0    0    -1
+$EndComp
+Text Label 4650 1950 2    60   ~ 0
+AC_Lout
+Text Label 5450 2400 2    60   ~ 0
+AC_Lout
 $EndSCHEMATC

Commit message: wireless-led: add first release
Parts:
- D1: symbol LED -> LED-RESCUE-light-node
- R1, R2, R3, R4, R5, R6, R7: symbol R -> R-RESCUE-light-node
- T1: symbol TRANSFO -> TRANSFO-RESCUE-light-node
Changed lines of the file:
@@
 EESchema Schematic File Version 2
+LIBS:light-node-rescue
 LIBS:power
 LIBS:device
@@
 LIBS:memory
 LIBS:xilinx
-LIBS:special
 LIBS:microcontrollers
 LIBS:dsp
@@
 LIBS:esp866_esp-12
 LIBS:light-node-cache
-EELAYER 27 0
+EELAYER 25 0
 EELAYER END
 $Descr A4 11693 8268
@@
 $EndComp
 $Comp
-L TRANSFO T1
+L TRANSFO-RESCUE-light-node T1
 U 1 1 569CE00E
 P 1900 1650
@@
 $EndComp
 $Comp
-L R R2
+L R-RESCUE-light-node R2
 U 1 1 569CE394
 P 4050 3000
@@
 $EndComp
 $Comp
-L R R3
+L R-RESCUE-light-node R3
 U 1 1 569CE3A3
 P 4050 3150
@@
 $EndComp
 $Comp
-L R R4
+L R-RESCUE-light-node R4
 U 1 1 569CE3B2
 P 4050 3300
@@
 $EndComp
 $Comp
-L R R5
+L R-RESCUE-light-node R5
 U 1 1 569CE3C1
 P 3650 2400
@@
 $EndComp
 $Comp
-L R R6
+L R-RESCUE-light-node R6
 U 1 1 569CE3D0
 P 3650 3650
@@
 $EndComp
 $Comp
-L R R7
+L R-RESCUE-light-node R7
 U 1 1 569CE3DF
 P 1300 2800
@@
 $EndComp
 $Comp
-L R R1
+L R-RESCUE-light-node R1
 U 1 1 569CE3FD
 P 1300 2600
@@
 $EndComp
 $Comp
-L LED D1
+L LED-RESCUE-light-node D1
 U 1 1 569CE42A
 P 4000 4000
